File: Hardware/Motor_Driver/Motor_Driver.kicad_sch (KiCad schematic)
At the start: 2 parts, among them U1 IR4301, U2 74AHC1G00

Commit message: Oppdaterte detaljene på schematicen
Parts:
- removed U1: IR4301, Package_DFN_QFN:Infineon_PQFN-22-15-4EP_6x5mm_P0.65mm, symbol Amplifier_Audio:IR4301
- removed U2: 74AHC1G00, symbol 74xGxx:74AHC1G00
Other:
- company: (none) -> Bachelor gruppe E41
- title: (none) -> Motor Driver for BLDC
